File: KiCAD/KZ80-SC1602.sch (KiCad schematic (older format))
At the start: 12 parts, among them J1 PC-8001 ext BUS, J2 I/O ADDR JP, J3 SC1602 LED Module, SW1 LCD LIGHT SW, U1 74HC138, U2 74HC04

Commit message: REV1基板ガーバーデータ出力
Parts:
- R1: value R_US -> 470
Changed lines of the file:
@@
 P 6450 2550
 F 0 "R1" H 6518 2596 50  0000 L CNN
-F 1 "R_US" H 6518 2505 50  0000 L CNN
+F 1 "470" H 6518 2505 50  0000 L CNN
 F 2 "" V 6490 2540 50  0001 C CNN
 F 3 "~" H 6450 2550 50  0001 C CNN
